Commit message: åæl

File: src/rudolph_v4/urdf/rudolph_v4.urdf (robot description, URDF)
Before this commit: robot rudolph_v4, 3 links, 2 joints
Joints:
- removed joint foot_print
- added joint base_footprint: type continuous, parent base_laser, child lidar_to_footprint, origin xyz=0 -0.184869976584764 0 rpy=0 0 0, axis 0.335999590456849 0 -0.941862131743723
